Commit message: hardware interface mods

File: protobot_description/urdf/control.xacro (robot description, xacro)
@@ -13,5 +13,5 @@
                 </hardware>
             </xacro:unless>
-            <joint name="shoulder_joint">
+            <joint name="shoulder">
                 <command_interface name="position">
                     <param name="min">-${(3*pi) / 4.0}</param>

File: protobot_description/urdf/gz.xacro (robot description, xacro)
@@ -6,5 +6,5 @@
             name="gz::sim::systems::JointStatePublisher">
             <topic>joint_states</topic>
-            <joint_name>shoulder_joint</joint_name>
+            <joint_name>shoulder</joint_name>
         </plugin>
     </gazebo>
@@ -13,5 +13,5 @@
             filename="gz-sim-joint-position-controller-system"
             name="gz::sim::systems::JointPositionController">
-            <joint_name>shoulder_joint</joint_name>
+            <joint_name>shoulder</joint_name>
             <p_gain>1</p_gain>
             <i_gain>0.1</i_gain>

File: protobot_description/urdf/structure.xacro (robot description, xacro)
@@ -55,5 +55,5 @@
         <child link="base_link" />
     </joint>
-    <joint name="shoulder_joint" type="revolute">
+    <joint name="shoulder" type="revolute">
         <origin xyz="0.03 0 0.28" rpy="0 0 0" />
         <parent link="base_link" />

Commit message: finaly pure pwm motor driver

File: protobot_description/urdf/control.xacro (robot description, xacro)
@@ -15,6 +15,6 @@
             <joint name="shoulder">
                 <command_interface name="position">
-                    <param name="min">-${(3*pi) / 4.0}</param>
-                    <param name="max">${(3*pi) / 4.0}</param>
+                    <param name="min">0.0</param>
+                    <param name="max">${(3*pi) / 2.0}</param>
                 </command_interface>
                 <state_interface name="position"/>

File: protobot_description/urdf/structure.xacro (robot description, xacro)
@@ -60,5 +60,5 @@
         <child link="upper_link" />
         <axis xyz="1 0 0" />
-        <limit lower="-${(3*pi)/4}" upper="${(3*pi)/4}" effort="10" velocity="1" />
+        <limit lower="0.0" upper="${(3*pi)/2}" effort="10" velocity="1" />
     </joint>
 </robot>
